Commit message: feat(C64,C65): Camera-Only 전환 + 상위 문서 정합성 갱신
C64: LiDAR 전면 제거, RGBD 카메라 ×3 전환
- model.sdf: rgbd_camera 센서 3대 (front/left/right)
- bridge_config.yaml: 카메라 RGB + PointCloud2 브릿지 6개 토픽
- nav2_params.yaml: obstacle_layer + collision_monitor PointCloud2 소스
- ss500.urdf.xacro: 카메라 3대 링크/조인트, LiDAR 제거
- simulation_launch.py: 카메라 frame bridge 3개
- perception_node.py: 멀티카메라 구독 전환
- ARCH-005 Camera-Only 인지 아키텍처 ADR 작성

C65: 상위 문서 C64 반영 + TASK 정합성 정리
- Application Definition: 센서 스펙, 인지 모듈, 구현 현황 갱신
- SYSTEM_OVERVIEW: 데이터 흐름도, TF 트리, costmap, ADR 인덱스
- TASK.md: C66~C69 신규 등록, C41 상태 갱신, C61 중복 정리

Co-Authored-By: Claude Opus 4.6 (1M context) <noreply@anthropic.com>

File: src/ad_bringup/urdf/ss500.urdf.xacro (robot description, xacro)
@@ -4,9 +4,13 @@
   TF 트리:
     base_footprint → base_link → imu_link
-                                → lidar_link
-                                → camera_link
+                                → camera_front_link
+                                → camera_left_link  (좌전방 ~60°)
+                                → camera_right_link (우전방 ~60°)
                                 → gps_link
                                 → left_track
                                 → right_track
+  센서 구성 (C64 확정, 2026-03-13):
+    카메라 3대 (전면 + 좌전방 60° + 우전방 60°), IMU, GPS
+    LiDAR 미탑재
 -->
 <robot xmlns:xacro="http://www.ros.org/wiki/xacro" name="ss500">
@@ -100,27 +104,4 @@
   </joint>
   <!-- ================================================================ -->
-  <!-- LiDAR -->
-  <!-- ================================================================ -->
-  <link name="lidar_link">
-    <visual>
-      <geometry>
-        <cylinder radius="0.05" length="0.08"/>
-      </geometry>
-      <material name="lidar_black">
-        <color rgba="0.15 0.15 0.15 1"/>
-      </material>
-    </visual>
-    <inertial>
-      <mass value="0.5"/>
-      <inertia ixx="0.001" iyy="0.001" izz="0.001"
-               ixy="0" ixz="0" iyz="0"/>
-    </inertial>
-  </link>
-  <joint name="lidar_joint" type="fixed">
-    <parent link="base_link"/>
-    <child link="lidar_link"/>
-    <origin xyz="0 0 0.5" rpy="0 0 0"/>
-  </joint>
-  <!-- ================================================================ -->
   <!-- IMU -->
   <!-- ================================================================ -->
@@ -138,7 +119,7 @@
   </joint>
   <!-- ================================================================ -->
-  <!-- Camera (전방) -->
-  <!-- ================================================================ -->
-  <link name="camera_link">
+  <!-- Camera: 전면 (0°) -->
+  <!-- ================================================================ -->
+  <link name="camera_front_link">
     <visual>
       <geometry>
@@ -155,8 +136,56 @@
     </inertial>
   </link>
-  <joint name="camera_joint" type="fixed">
-    <parent link="base_link"/>
-    <child link="camera_link"/>
+  <joint name="camera_front_joint" type="fixed">
+    <parent link="base_link"/>
+    <child link="camera_front_link"/>
     <origin xyz="0.9 0 0.3" rpy="0 0 0"/>
+  </joint>
+  <!-- ================================================================ -->
+  <!-- Camera: 좌전방 (~60°) -->
+  <!-- ================================================================ -->
+  <link name="camera_left_link">
+    <visual>
+      <geometry>
+        <box size="0.05 0.08 0.05"/>
+      </geometry>
+      <material name="camera_black">
+        <color rgba="0.1 0.1 0.1 1"/>
+      </material>
+    </visual>
+    <inertial>
+      <mass value="0.2"/>
+      <inertia ixx="0.0002" iyy="0.0002" izz="0.0002"
+               ixy="0" ixz="0" iyz="0"/>
+    </inertial>
+  </link>
+  <joint name="camera_left_joint" type="fixed">
+    <parent link="base_link"/>
+    <child link="camera_left_link"/>
+    <!-- 차체 좌전방 모서리, yaw +60° (1.047 rad) -->
+    <origin xyz="0.7 0.5 0.3" rpy="0 0 1.047"/>
+  </joint>
+  <!-- ================================================================ -->
+  <!-- Camera: 우전방 (~60°) -->
+  <!-- ================================================================ -->
+  <link name="camera_right_link">
+    <visual>
+      <geometry>
+        <box size="0.05 0.08 0.05"/>
+      </geometry>
+      <material name="camera_black">
+        <color rgba="0.1 0.1 0.1 1"/>
+      </material>
+    </visual>
+    <inertial>
+      <mass value="0.2"/>
+      <inertia ixx="0.0002" iyy="0.0002" izz="0.0002"
+               ixy="0" ixz="0" iyz="0"/>
+    </inertial>
+  </link>
+  <joint name="camera_right_joint" type="fixed">
+    <parent link="base_link"/>
+    <child link="camera_right_link"/>
+    <!-- 차체 우전방 모서리, yaw -60° (-1.047 rad) -->
+    <origin xyz="0.7 -0.5 0.3" rpy="0 0 -1.047"/>
   </joint>
   <!-- ================================================================ -->
